Commit message: Add linearized Cart. Update installation guide

File: Projects/00_Cart/cart_vis/cart.urdf (robot description, URDF)
Before this commit: robot cart, 7 links, 6 joints
Links:
- link chassis: mass 6.0 -> 2.0
- link wheel_1: mass 1.0 -> 0.25
- link wheel_2: mass 1.0 -> 0.25
- link wheel_3: mass 1.0 -> 0.25
- link wheel_4: mass 1.0 -> 0.25
